File: clock-module.kicad_sch (KiCad schematic)
At the start: 14 parts, among them SW1 SW_SPDT, SW2 SW_Push, U1 SN74LS04N, U2 SN74LS08N

Commit message: Fix 74LS04N model and clock module simulation
Parts:
- removed R9: 10k, symbol Device:R
- removed unit 2 of U1
- added R4: 1M, symbol Device:R
- added unit 1 of U1
- S1, S2, V2, V3: now left out of the parts list
- renumbered R4 to R5
Connections:
- net CLK: now also U1.3; no longer U1.5
- net GND: now also R4.2
- net HALT: now also U1.1
- net ~{CLK}: now also U1.4, R4.1; no longer U1.6
- net ~{MAIN_CLK_EN}: now also S2.2 (N-); no longer S1.1 (N+)
- net ~{MANUAL_CLK_EN}: now also S1.1 (N+); no longer S2.2 (N-)
- net at U2.9: now also U1.2
