File: clock-selector.kicad_sch (KiCad schematic)
At the start: 5 parts, among them U1 SN74LS04N, U2 SN74LS08N, U5 NE555P, U6 HD74LS32P

Commit message: Fix 74LS04N model and clock module simulation
Parts:
- removed unit 1 of U1
- added R10: 1M, symbol Device:R
- added unit 3 of U1
Connections:
- net CLK: now also R10.1
- net CLK_SELECT: now also U1.5
- net GND: now also R10.2
- net at U2.2: now also U1.6
Other:
- moved on the sheet: C5
