File: main-clock.kicad_sch (KiCad schematic)
At the start: 6 parts, among them U4 NE555P

Commit message: Fix 74LS04N model and clock module simulation
Parts:
- renumbered R6 to R7, R7 to R8, R8 to R9
Changed lines of the file:
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@@
 		(dnp no)
 		(fields_autoplaced yes)
-		(property "Reference" "R8"
+		(property "Reference" "R9"
 			(at 193.04 86.3599 0)
 			(effects
@@
 			(project "8-bit-computer"
 				(path "/64f7f61e-1043-4516-89cf-db6a25fcb096/9534564d-2813-40f9-953b-2838250e65d7/e503b9eb-d113-495b-825f-b3db55a219d0"
-					(reference "R8")
+					(reference "R9")
 					(unit 1)
 				)
@@
 		(dnp no)
 		(fields_autoplaced yes)
-		(property "Reference" "R6"
+		(property "Reference" "R7"
 			(at 173.99 69.8499 0)
 			(effects
@@
 			(project "8-bit-computer"
 				(path "/64f7f61e-1043-4516-89cf-db6a25fcb096/9534564d-2813-40f9-953b-2838250e65d7/e503b9eb-d113-495b-825f-b3db55a219d0"
-					(reference "R6")
+					(reference "R7")
 					(unit 1)
 				)
@@
 		(dnp no)
 		(fields_autoplaced yes)
-		(property "Reference" "R7"
+		(property "Reference" "R8"
 			(at 180.34 74.93 90)
 			(effects
@@
 			(project "8-bit-computer"
 				(path "/64f7f61e-1043-4516-89cf-db6a25fcb096/9534564d-2813-40f9-953b-2838250e65d7/e503b9eb-d113-495b-825f-b3db55a219d0"
-					(reference "R7")
+					(reference "R8")
 					(unit 1)
 				)
