File: manual-clock.kicad_sch (KiCad schematic)
At the start: 4 parts, among them U3 NE555P

Commit message: Fix 74LS04N model and clock module simulation
Parts:
- renumbered R5 to R6
Changed lines of the file:
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@@
 		(dnp no)
 		(fields_autoplaced yes)
-		(property "Reference" "R5"
+		(property "Reference" "R6"
 			(at 154.94 62.2299 0)
 			(effects
@@
 			(project "8-bit-computer"
 				(path "/64f7f61e-1043-4516-89cf-db6a25fcb096/9534564d-2813-40f9-953b-2838250e65d7/8b8c0dd5-63d2-4989-a35c-f894197311aa"
-					(reference "R5")
+					(reference "R6")
 					(unit 1)
 				)
